File: transmitter.sch (EAGLE design)
At the start: 25 parts, among them IC1 MEGA8-AI, X1 ARK-3.5MMAPC2, X2 ARK-3.5MMAPC2, X3 ARK-3.5MMAPC2

Commit message: usuniecie masy, przestawienie led, wiekszy opis
Parts:
- C8, C9: value 100nF -> 10nF
- R6, R7: value 1k -> 100
Changed lines of the file:
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@@
 <part name="R3" library="rcl" library_urn="urn:adsk.eagle:library:334" deviceset="R-EU_" device="M0805" package3d_urn="urn:adsk.eagle:package:23556/2" value="100k"/>
 <part name="C7" library="rcl" library_urn="urn:adsk.eagle:library:334" deviceset="C-EU" device="C0805" package3d_urn="urn:adsk.eagle:package:23617/2" value="100nF"/>
-<part name="R6" library="rcl" library_urn="urn:adsk.eagle:library:334" deviceset="R-EU_" device="M0805" package3d_urn="urn:adsk.eagle:package:23556/2" value="1k"/>
-<part name="R7" library="rcl" library_urn="urn:adsk.eagle:library:334" deviceset="R-EU_" device="M0805" package3d_urn="urn:adsk.eagle:package:23556/2" value="1k"/>
-<part name="C8" library="rcl" library_urn="urn:adsk.eagle:library:334" deviceset="C-EU" device="C0805" package3d_urn="urn:adsk.eagle:package:23617/2" value="100nF"/>
-<part name="C9" library="rcl" library_urn="urn:adsk.eagle:library:334" deviceset="C-EU" device="C0805" package3d_urn="urn:adsk.eagle:package:23617/2" value="100nF"/>
+<part name="R6" library="rcl" library_urn="urn:adsk.eagle:library:334" deviceset="R-EU_" device="M0805" package3d_urn="urn:adsk.eagle:package:23556/2" value="100"/>
+<part name="R7" library="rcl" library_urn="urn:adsk.eagle:library:334" deviceset="R-EU_" device="M0805" package3d_urn="urn:adsk.eagle:package:23556/2" value="100"/>
+<part name="C8" library="rcl" library_urn="urn:adsk.eagle:library:334" deviceset="C-EU" device="C0805" package3d_urn="urn:adsk.eagle:package:23617/2" value="10nF"/>
+<part name="C9" library="rcl" library_urn="urn:adsk.eagle:library:334" deviceset="C-EU" device="C0805" package3d_urn="urn:adsk.eagle:package:23617/2" value="10nF"/>
 <part name="GND3" library="supply1" library_urn="urn:adsk.eagle:library:371" deviceset="GND" device=""/>
 <part name="GND6" library="supply1" library_urn="urn:adsk.eagle:library:371" deviceset="GND" device=""/>

Commit message: drobne poprawki
Parts:
- added S1: REED-SWITCH-MK6-6, switch-reed:REED-SWITCH-MK6-6
- renumbered LED1 to LED
Connections:
- removed net SWITCH2_WIRE: R6.2, X2-1.K
- new net N$3: R6.2, S1.2, X2-2.K
- net GND: now also S1.1, X2-1.K; no longer X2-2.K
Other:
- moved on the sheet: X2-1, X2-2
Changed lines of the file:
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@@
 <part name="GND5" library="supply1" library_urn="urn:adsk.eagle:library:371" deviceset="GND" device=""/>
 <part name="+3V6" library="supply1" library_urn="urn:adsk.eagle:library:371" deviceset="+3V3" device=""/>
-<part name="X1" library="Connectors" deviceset="ARK-3.5MM" device="APC2" package3d_urn="urn:adsk.eagle:package:24782377/4"/>
-<part name="X2" library="Connectors" deviceset="ARK-3.5MM" device="APC2" package3d_urn="urn:adsk.eagle:package:24782377/4"/>
-<part name="X3" library="Connectors" deviceset="ARK-3.5MM" device="APC2" package3d_urn="urn:adsk.eagle:package:24782377/4"/>
+<part name="X1" library="Connectors" library_urn="urn:adsk.eagle:library:25621963" deviceset="ARK-3.5MM" device="APC2" package3d_urn="urn:adsk.eagle:package:24782377/5"/>
+<part name="X2" library="Connectors" library_urn="urn:adsk.eagle:library:25621963" deviceset="ARK-3.5MM" device="APC2" package3d_urn="urn:adsk.eagle:package:24782377/5"/>
+<part name="X3" library="Connectors" library_urn="urn:adsk.eagle:library:25621963" deviceset="ARK-3.5MM" device="APC2" package3d_urn="urn:adsk.eagle:package:24782377/5"/>
 <part name="U$1" library="Modules" deviceset="NRF24L01+" device="" package3d_urn="urn:adsk.eagle:package:24547223/3"/>
 <part name="GND8" library="supply1" library_urn="urn:adsk.eagle:library:371" deviceset="GND" device=""/>
@@
 <part name="R4" library="rcl" library_urn="urn:adsk.eagle:library:334" deviceset="R-EU_" device="M0805" package3d_urn="urn:adsk.eagle:package:23556/2" value="4.7M"/>
 <part name="GND7" library="supply1" library_urn="urn:adsk.eagle:library:371" deviceset="GND" device=""/>
-<part name="DC3-ISP" library="Connectors" deviceset="ML10" device="" package3d_urn="urn:adsk.eagle:package:24836372/3"/>
-<part name="JP1" library="Connectors" deviceset="PINHD-1X1" device="" package3d_urn="urn:adsk.eagle:package:22485/2"/>
-<part name="LED1" library="led" library_urn="urn:adsk.eagle:library:259" deviceset="LED" device="CHIP-LED0805" package3d_urn="urn:adsk.eagle:package:15818/2"/>
+<part name="DC3-ISP" library="Connectors" library_urn="urn:adsk.eagle:library:25621963" deviceset="ML10" device="" package3d_urn="urn:adsk.eagle:package:24836372/3"/>
+<part name="JP1" library="Connectors" library_urn="urn:adsk.eagle:library:25621963" deviceset="PINHD-1X1" device="" package3d_urn="urn:adsk.eagle:package:25621971/1"/>
+<part name="LED" library="led" library_urn="urn:adsk.eagle:library:259" deviceset="LED" device="CHIP-LED0805" package3d_urn="urn:adsk.eagle:package:15818/2"/>
 <part name="+3V1" library="supply1" library_urn="urn:adsk.eagle:library:371" deviceset="+3V3" device=""/>
 <part name="R8" library="rcl" library_urn="urn:adsk.eagle:library:334" deviceset="R-EU_" device="M0805" package3d_urn="urn:adsk.eagle:package:23556/2" value="10"/>
 <part name="S2" library="Modules" deviceset="TS-1187A-B-A-B" device="" package3d_urn="urn:adsk.eagle:package:24754950/2"/>
+<part name="S1" library="switch-reed" deviceset="REED-SWITCH-" device="MK6-6" package3d_urn="urn:adsk.eagle:package:27523/1"/>
 </parts>
 <sheets>
@@
 <attribute name="NAME" x="135.89" y="-3.429" size="1.778" layer="95"/>
 </instance>
-<instance part="X2" gate="-1" x="190.5" y="15.24" smashed="yes">
-<attribute name="NAME" x="191.77" y="14.351" size="1.778" layer="95"/>
-</instance>
-<instance part="X2" gate="-2" x="190.5" y="-2.54" smashed="yes">
-<attribute name="NAME" x="191.77" y="-3.429" size="1.778" layer="95"/>
+<instance part="X2" gate="-1" x="193.04" y="-2.54" smashed="yes">
+<attribute name="NAME" x="194.31" y="-3.429" size="1.778" layer="95"/>
+</instance>
+<instance part="X2" gate="-2" x="193.04" y="15.24" smashed="yes">
+<attribute name="NAME" x="194.31" y="14.351" size="1.778" layer="95"/>
 </instance>
 <instance part="X3" gate="-1" x="-30.48" y="86.36" smashed="yes" rot="MR0">
@@
 <attribute name="VALUE" x="46.99" y="63.5" size="1.778" layer="96"/>
 </instance>
-<instance part="LED1" gate="G$1" x="43.18" y="114.3" smashed="yes">
+<instance part="LED" gate="G$1" x="43.18" y="114.3" smashed="yes">
 <attribute name="NAME" x="46.736" y="109.728" size="1.778" layer="95" rot="R90"/>
 <attribute name="VALUE" x="48.895" y="109.728" size="1.778" layer="96" rot="R90"/>
@@
 <attribute name="NAME" x="134.62" y="-25.4" size="1.27" layer="95"/>
 <attribute name="VALUE" x="134.62" y="-30.48" size="1.27" layer="96" align="top-left"/>
+</instance>
+<instance part="S1" gate="G$1" x="187.96" y="7.62" smashed="yes" rot="R180">
+<attribute name="NAME" x="190.5" y="2.54" size="1.778" layer="95"/>
 </instance>
 </instances>
@@
 <segment>
 <pinref part="+3V1" gate="G$1" pin="+3V3"/>
-<pinref part="LED1" gate="G$1" pin="A"/>
+<pinref part="LED" gate="G$1" pin="A"/>
 <wire x1="43.18" y1="116.84" x2="43.18" y2="121.92" width="0.1524" layer="91"/>
 </segment>
@@
 <pinref part="C8" gate="G$1" pin="1"/>
 <wire x1="170.18" y1="-5.08" x2="170.18" y2="-2.54" width="0.1524" layer="91"/>
-<pinref part="X2" gate="-2" pin="K"/>
 <wire x1="170.18" y1="-2.54" x2="170.18" y2="2.54" width="0.1524" layer="91"/>
-<wire x1="187.96" y1="-2.54" x2="175.26" y2="-2.54" width="0.1524" layer="91"/>
 <junction x="170.18" y="-2.54"/>
 <pinref part="R4" gate="G$1" pin="1"/>
-<wire x1="175.26" y1="-2.54" x2="170.18" y2="-2.54" width="0.1524" layer="91"/>
 <wire x1="170.18" y1="-2.54" x2="175.26" y2="-2.54" width="0.1524" layer="91"/>
 <wire x1="175.26" y1="-2.54" x2="175.26" y2="0" width="0.1524" layer="91"/>
+<pinref part="X2" gate="-1" pin="K"/>
+<wire x1="175.26" y1="-2.54" x2="187.96" y2="-2.54" width="0.1524" layer="91"/>
 <junction x="175.26" y="-2.54"/>
+<pinref part="S1" gate="G$1" pin="1"/>
+<wire x1="187.96" y1="-2.54" x2="190.5" y2="-2.54" width="0.1524" layer="91"/>
+<wire x1="187.96" y1="-2.54" x2="187.96" y2="0" width="0.1524" layer="91"/>
+<junction x="187.96" y="-2.54"/>
 </segment>
 <segment>
@@
 <wire x1="-45.72" y1="15.24" x2="-35.56" y2="15.24" width="0.1524" layer="91"/>
 <junction x="-35.56" y="15.24"/>
-</segment>
-</net>
-<net name="SWITCH2_WIRE" class="0">
-<segment>
-<pinref part="X2" gate="-1" pin="K"/>
-<pinref part="R6" gate="G$1" pin="2"/>
-<wire x1="185.42" y1="15.24" x2="187.96" y2="15.24" width="0.1524" layer="91"/>
 </segment>
 </net>
@@
 <net name="N$2" class="0">
 <segment>
-<pinref part="LED1" gate="G$1" pin="C"/>
+<pinref part="LED" gate="G$1" pin="C"/>
 <pinref part="R8" gate="G$1" pin="2"/>
 <wire x1="43.18" y1="106.68" x2="43.18" y2="109.22" width="0.1524" layer="91"/>
 </segment>
 </net>
+<net name="N$3" class="0">
+<segment>
+<pinref part="R6" gate="G$1" pin="2"/>
+<pinref part="X2" gate="-2" pin="K"/>
+<wire x1="185.42" y1="15.24" x2="187.96" y2="15.24" width="0.1524" layer="91"/>
+<pinref part="S1" gate="G$1" pin="2"/>
+<wire x1="187.96" y1="15.24" x2="190.5" y2="15.24" width="0.1524" layer="91"/>
+<wire x1="187.96" y1="12.7" x2="187.96" y2="15.24" width="0.1524" layer="91"/>
+<junction x="187.96" y="15.24"/>
+</segment>
+</net>
